Commit message: updated colors

File: urdf/_d435.gazebo.xacro (robot description, xacro)
@@ -6,8 +6,10 @@
 -->
 <robot xmlns:xacro="http://ros.org/wiki/xacro">
+  <xacro:property name="skyblue" value="Gazebo/BlueGlow" />
   <xacro:macro name="gazebo_d435" params="camera_name reference_link topics_ns depth_optical_frame color_optical_frame infrared1_optical_frame infrared2_optical_frame" >
     <!-- Load parameters to model's main link-->
     <xacro:property name="deg_to_rad" value="0.01745329251994329577" />
     <gazebo reference="${reference_link}">
+      <material>${skyblue}</material>
       <self_collide>0</self_collide>
       <enable_wind>0</enable_wind>
